File: PCB2/BacklitBadge2/schematic.brd (EAGLE design)
At the start: 80 x 100 mm, 35 parts

Commit message: Updates to the schematic
Parts:
- added C1, C2: (no value), eagle-ltspice:C1206
- moved R4 91.7 mm to (5.00, 81.0), turned to 270 degrees
- moved R5 90.7 mm to (5.00, 75.0), turned to 90 degrees
- moved R6 89.7 mm to (5.00, 69.0), turned to 270 degrees
- turned LED2 to 270 degrees
- turned LED3 to 90 degrees
Connections:
- removed net N$30: R5.2, U$2.P$4
- new net N$9: LED3.C, R6.2
- net CHRG_IN: now also C1.1, LED1.A, LED2.A, LED3.A
- net GND: now also C1.2, C2.2; no longer LED1.C, LED2.C, LED3.C
- net N$14: now also R5.1, U$2.P$4; no longer LED1.A, R4.1
- net N$28: now also R4.1; no longer R6.2
- net N$6: now also LED1.C, R4.2; no longer LED3.A, R6.1
- net N$7: now also LED2.C, R5.2; no longer LED2.A, R5.1
- net N$8: now also R6.1; no longer R4.2
- net VCC: now also C2.1
